Commit message: augmented lagrangian prototype

File: models/biped/urdf/biped_float.urdf (robot description, URDF)
Before this commit: robot flip_5link, 8 links, 7 joints
Links:
- link left_shank: geometry visual GeometryTypes.Sphere radius=0.02; visual cylinder length=0.288 radius=0.02
- link right_shank: geometry visual GeometryTypes.Sphere radius=0.02; visual cylinder length=0.288 radius=0.02

File: models/biped/urdf/biped_left_pinned.urdf (robot description, URDF)
Before this commit: robot flip_5link, 6 links, 5 joints
Links:
- link left_shank: geometry visual GeometryTypes.Sphere radius=0.02; visual cylinder length=0.288 radius=0.02
- link right_shank: geometry visual GeometryTypes.Sphere radius=0.02; visual cylinder length=0.288 radius=0.02

File: models/biped/urdf/biped_right_pinned.urdf (robot description, URDF)
Before this commit: robot flip_5link, 6 links, 5 joints
Links:
- link left_shank: geometry visual GeometryTypes.Sphere radius=0.02; visual cylinder length=0.288 radius=0.02
- link right_shank: geometry visual GeometryTypes.Sphere radius=0.02; visual cylinder length=0.288 radius=0.02

Commit message: simulate box drop

File: models/biped/urdf/biped_float.urdf (robot description, URDF)
Before this commit: robot flip_5link, 8 links, 7 joints
Links:
- link left_shank: geometry visual Sphere radius=0.02; visual cylinder length=0.288 radius=0.02
- link right_shank: geometry visual Sphere radius=0.02; visual cylinder length=0.288 radius=0.02

File: models/biped/urdf/biped_left_pinned.urdf (robot description, URDF)
Before this commit: robot flip_5link, 6 links, 5 joints
Links:
- link left_shank: geometry visual Sphere radius=0.02; visual cylinder length=0.288 radius=0.02
- link right_shank: geometry visual Sphere radius=0.02; visual cylinder length=0.288 radius=0.02

File: models/biped/urdf/biped_right_pinned.urdf (robot description, URDF)
Before this commit: robot flip_5link, 6 links, 5 joints
Links:
- link left_shank: geometry visual Sphere radius=0.02; visual cylinder length=0.288 radius=0.02
- link right_shank: geometry visual Sphere radius=0.02; visual cylinder length=0.288 radius=0.02
