Commit message: methods for including model, obj, con

File: models/kuka/temp/kuka.urdf (robot description, URDF)
Before this commit: robot iiwa14, 11 links, 10 joints
Links:
- link iiwa_link_0: geometry visual mesh filename=/home/taylor/.julia/dev/DirectMotionPlanning/models/kuka/me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
- link iiwa_link_1: geometry visual mesh filename=/home/taylor/.julia/dev/DirectMotionPlanning/models/kuka/me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
- link iiwa_link_2: geometry visual mesh filename=/home/taylor/.julia/dev/DirectMotionPlanning/models/kuka/me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
- link iiwa_link_3: geometry visual mesh filename=/home/taylor/.julia/dev/DirectMotionPlanning/models/kuka/me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
- link iiwa_link_4: geometry visual mesh filename=/home/taylor/.julia/dev/DirectMotionPlanning/models/kuka/me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
- link iiwa_link_5: geometry visual mesh filename=/home/taylor/.julia/dev/DirectMotionPlanning/models/kuka/me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
- link iiwa_link_6: geometry visual mesh filename=/home/taylor/.julia/dev/DirectMotionPlanning/models/kuka/me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
- link iiwa_link_7: geometry collision mesh filename=/home/taylor/.julia/dev/DirectMotionPlanning/models/kuka/me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; visual mesh filename=/home/taylor/.julia/dev/DirectMotionPlanning/models/kuka/me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

Commit message: motion_planning

File: models/kuka/temp/kuka.urdf (robot description, URDF)
Before this commit: robot iiwa14, 11 links, 10 joints
Links:
- link iiwa_link_0: geometry visual mesh filename=/home/taylor/.julia/dev/motion_planning/models/kuka/meshes/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
- link iiwa_link_1: geometry visual mesh filename=/home/taylor/.julia/dev/motion_planning/models/kuka/meshes/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
- link iiwa_link_2: geometry visual mesh filename=/home/taylor/.julia/dev/motion_planning/models/kuka/meshes/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
- link iiwa_link_3: geometry visual mesh filename=/home/taylor/.julia/dev/motion_planning/models/kuka/meshes/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
- link iiwa_link_4: geometry visual mesh filename=/home/taylor/.julia/dev/motion_planning/models/kuka/meshes/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
- link iiwa_link_5: geometry visual mesh filename=/home/taylor/.julia/dev/motion_planning/models/kuka/meshes/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
- link iiwa_link_6: geometry visual mesh filename=/home/taylor/.julia/dev/motion_planning/models/kuka/meshes/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
- link iiwa_link_7: geometry collision mesh filename=/home/taylor/.julia/dev/motion_planning/models/kuka/meshes/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; visual mesh filename=/home/taylor/.julia/dev/motion_planning/models/kuka/meshes/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
